File: pcb/macropad.kicad_pcb (KiCad board)
At the start: 2 copper layers, 61.9 x 83.3 mm, 21 parts, among them U1 Seeeduino Xiao rp2040

Commit message: added silkscreen
Parts:
- moved G*** 67.8 mm to (174.8, 133.4)
Changed lines of the file:
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@@
 	(footprint "LOGO"
 		(layer "B.Cu")
-		(at 173.595094 65.612113 180)
+		(at 174.785094 133.382113 180)
 		(property "Reference" "G***"
 			(at 0 0 0)
@@
 	)
 	(gr_text "Macropad v0.1"
-		(at 185.14 76.2125 0)
+		(at 168.68 82.1925 0)
 		(layer "B.SilkS")
 		(effects
@@
 		)
 	)
+	(barcode
+		(at 158.067726 69.260932 0)
+		(layer "B.SilkS")
+		(size 13.735702 13.735702)
+		(text "https://github.com/poggersv2/macropad")
+		(text_height 0.5)
+		(type qr)
+		(ecc_level L)
+		(hide no)
+		(knockout no)
+	)
 	(segment

Commit message: Added fill zones
Routing:
- added copper zone on B.Cu, net GND
- added copper zone on F.Cu, net GND
Changed lines of the file:
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@@
 		(tags "rotary encoder")
 		(property "Reference" "MX1"
-			(at 5.75 -6.999999 90)
+			(at 9.525 9.525 0)
 			(layer "F.SilkS")
+			(hide yes)
 			(effects
 				(font
@@
 	)
 	(segment
+		(start 176.487499 75.5825)
+		(end 146.89 75.5825)
+		(width 0.2)
+		(layer "F.Cu")
+		(net "ROTSW")
+	)
+	(segment
+		(start 182.895 69.174999)
+		(end 176.487499 75.5825)
+		(width 0.2)
+		(layer "F.Cu")
+		(net "ROTSW")
+	)
+	(segment
 		(start 141.795 105.9175)
 		(end 146.02 105.9175)
@@
 		(net "Net-(D5-A)")
 	)
-	(segment
-		(start 176.487499 75.5825)
-		(end 146.89 75.5825)
-		(width 0.2)
+	(zone
+		(net "GND")
 		(layer "F.Cu")
-		(net "ROTSW")
+		(hatch edge 0.5)
+		(connect_pads
+			(clearance 0.5)
+		)
+		(min_thickness 0.25)
+		(fill yes
+			(thermal_gap 0.5)
+			(thermal_bridge_width 0.5)
+			(island_removal_mode 0)
+		)
+		(polygon
+			(pts
+				(xy 118.745 52.3875) (xy 194.945 52.3875) (xy 194.945 147.6375) (xy 118.745 147.6375)
+			)
+		)
 	)
-	(segment
-		(start 182.895 69.174999)
-		(end 176.487499 75.5825)
-		(width 0.2)
-		(layer "F.Cu")
-		(net "ROTSW")
+	(zone
+		(net "GND")
+		(layer "B.Cu")
+		(hatch edge 0.5)
+		(priority 1)
+		(connect_pads
+			(clearance 0.5)
+		)
+		(min_thickness 0.25)
+		(fill yes
+			(thermal_gap 0.5)
+			(thermal_bridge_width 0.5)
+			(island_removal_mode 0)
+		)
+		(polygon
+			(pts
+				(xy 118.745 52.3875) (xy 194.945 52.3875) (xy 194.945 147.6375) (xy 118.745 147.6375)
+			)
+		)
 	)
 	(embedded_fonts no)
